File: Control stepper/Control stepper.kicad_pcb (KiCad board)
At the start: 2 copper layers, 12 parts, among them J1 Conn_01x04, J2 Conn_01x02, J3 Conn_01x03, Q1 2n2222a, Q2 2n2222a, Q3 2n2222a, Q4 2n2222a, U1 4017

Commit message: final
Parts:
- removed the J1 at (181.6, 68.6)
- removed the J2 at (121.9, 77.5)
- removed the J3 at (129.5, 54.6)
- removed the Q1 at (168.9, 66.0)
- removed the Q2 at (168.9, 72.4)
- removed the Q3 at (168.9, 80.0)
- removed the Q4 at (168.9, 86.4)
- removed the R1 at (146.1, 86.4)
- removed the R2 at (146.1, 80.0)
- removed the R3 at (162.6, 68.6)
- removed the R4 at (162.6, 62.2)
- removed the U1 at (138.4, 83.8)
- added J1: Conn_01x04, TerminalBlock:TerminalBlock_bornier-4_P5.08mm, F.Cu at (172.9, 75.6)
- added J1: Conn_01x04, TerminalBlock:TerminalBlock_bornier-4_P5.08mm, F.Cu at (87.0, 117.7)
- added J1: Conn_01x04, TerminalBlock:TerminalBlock_bornier-4_P5.08mm, F.Cu at (257.2, 74.5)
- added J1: Conn_01x04, TerminalBlock:TerminalBlock_bornier-4_P5.08mm, F.Cu at (258.7, 31.1)
- added J1: Conn_01x04, TerminalBlock:TerminalBlock_bornier-4_P5.08mm, F.Cu at (172.5, 118.1)
- added J1: Conn_01x04, TerminalBlock:TerminalBlock_bornier-4_P5.08mm, F.Cu at (167.9, 166.6)
- added J1: Conn_01x04, TerminalBlock:TerminalBlock_bornier-4_P5.08mm, F.Cu at (87.0, 75.3)
- added J1: Conn_01x04, TerminalBlock:TerminalBlock_bornier-4_P5.08mm, F.Cu at (85.9, 164.5)
- added J1: Conn_01x04, TerminalBlock:TerminalBlock_bornier-4_P5.08mm, F.Cu at (87.0, 31.4)
- added J1: Conn_01x04, TerminalBlock:TerminalBlock_bornier-4_P5.08mm, F.Cu at (173.3, 32.2)
- added J1: Conn_01x04, TerminalBlock:TerminalBlock_bornier-4_P5.08mm, F.Cu at (258.4, 117.3)
- added J2: Conn_01x02, TerminalBlock:TerminalBlock_bornier-2_P5.08mm, F.Cu at (204.3, 110.4)
- added J2: Conn_01x02, TerminalBlock:TerminalBlock_bornier-2_P5.08mm, F.Cu at (203.2, 67.6)
- added J2: Conn_01x02, TerminalBlock:TerminalBlock_bornier-2_P5.08mm, F.Cu at (119.3, 25.3)
- added J2: Conn_01x02, TerminalBlock:TerminalBlock_bornier-2_P5.08mm, F.Cu at (33.0, 68.3)
- added J2: Conn_01x02, TerminalBlock:TerminalBlock_bornier-2_P5.08mm, F.Cu at (31.9, 157.6)
- added J2: Conn_01x02, TerminalBlock:TerminalBlock_bornier-2_P5.08mm, F.Cu at (118.9, 68.7)
- added J2: Conn_01x02, TerminalBlock:TerminalBlock_bornier-2_P5.08mm, F.Cu at (33.0, 24.5)
- added J2: Conn_01x02, TerminalBlock:TerminalBlock_bornier-2_P5.08mm, F.Cu at (113.9, 159.6)
- added J2: Conn_01x02, TerminalBlock:TerminalBlock_bornier-2_P5.08mm, F.Cu at (118.5, 111.1)
- added J2: Conn_01x02, TerminalBlock:TerminalBlock_bornier-2_P5.08mm, F.Cu at (204.7, 24.1)
- added J2: Conn_01x02, TerminalBlock:TerminalBlock_bornier-2_P5.08mm, F.Cu at (33.0, 110.7)
- added J3: Conn_01x03, TerminalBlock:TerminalBlock_bornier-3_P5.08mm, F.Cu at (25.4, 37.2)
- added J3: Conn_01x03, TerminalBlock:TerminalBlock_bornier-3_P5.08mm, F.Cu at (110.9, 123.8)
- added J3: Conn_01x03, TerminalBlock:TerminalBlock_bornier-3_P5.08mm, F.Cu at (106.3, 172.3)
- added J3: Conn_01x03, TerminalBlock:TerminalBlock_bornier-3_P5.08mm, F.Cu at (25.4, 123.4)
- added J3: Conn_01x03, TerminalBlock:TerminalBlock_bornier-3_P5.08mm, F.Cu at (25.4, 81.0)
- added J3: Conn_01x03, TerminalBlock:TerminalBlock_bornier-3_P5.08mm, F.Cu at (195.6, 80.3)
- added J3: Conn_01x03, TerminalBlock:TerminalBlock_bornier-3_P5.08mm, F.Cu at (111.6, 38.0)
- added J3: Conn_01x03, TerminalBlock:TerminalBlock_bornier-3_P5.08mm, F.Cu at (197.1, 36.8)
- added J3: Conn_01x03, TerminalBlock:TerminalBlock_bornier-3_P5.08mm, F.Cu at (111.3, 81.4)
- added J3: Conn_01x03, TerminalBlock:TerminalBlock_bornier-3_P5.08mm, F.Cu at (24.3, 170.3)
- added J3: Conn_01x03, TerminalBlock:TerminalBlock_bornier-3_P5.08mm, F.Cu at (196.7, 123.1)
- added Q1: 2N3904BU, Package_TO_SOT_THT:TO-92, F.Cu at (74.3, 115.1)
- added Q1: 2N3904BU, Package_TO_SOT_THT:TO-92, F.Cu at (246.0, 28.5)
- added Q1: 2N3904BU, Package_TO_SOT_THT:TO-92, F.Cu at (159.8, 115.5)
- added Q1: 2N3904BU, Package_TO_SOT_THT:TO-92, F.Cu at (74.3, 72.7)
- added Q1: 2N3904BU, Package_TO_SOT_THT:TO-92, F.Cu at (73.2, 162.0)
- added Q1: 2N3904BU, Package_TO_SOT_THT:TO-92, F.Cu at (244.5, 72.0)
- added Q1: 2N3904BU, Package_TO_SOT_THT:TO-92, F.Cu at (160.6, 29.7)
- added Q1: 2N3904BU, Package_TO_SOT_THT:TO-92, F.Cu at (155.2, 164.0)
- added Q1: 2N3904BU, Package_TO_SOT_THT:TO-92, F.Cu at (160.2, 73.1)
- added Q1: 2N3904BU, Package_TO_SOT_THT:TO-92, F.Cu at (74.3, 28.9)
- added Q1: 2N3904BU, Package_TO_SOT_THT:TO-92, F.Cu at (245.7, 114.8)
- added Q2: 2N3904BU, Package_TO_SOT_THT:TO-92, F.Cu at (160.2, 80.7)
- added Q2: 2N3904BU, Package_TO_SOT_THT:TO-92, F.Cu at (160.6, 37.3)
- added Q2: 2N3904BU, Package_TO_SOT_THT:TO-92, F.Cu at (159.8, 123.1)
- added Q2: 2N3904BU, Package_TO_SOT_THT:TO-92, F.Cu at (244.5, 79.6)
- added Q2: 2N3904BU, Package_TO_SOT_THT:TO-92, F.Cu at (74.3, 122.8)
- added Q2: 2N3904BU, Package_TO_SOT_THT:TO-92, F.Cu at (246.0, 36.1)
- added Q2: 2N3904BU, Package_TO_SOT_THT:TO-92, F.Cu at (73.2, 169.6)
- added Q2: 2N3904BU, Package_TO_SOT_THT:TO-92, F.Cu at (155.2, 171.6)
- added Q2: 2N3904BU, Package_TO_SOT_THT:TO-92, F.Cu at (74.3, 80.3)
- added Q2: 2N3904BU, Package_TO_SOT_THT:TO-92, F.Cu at (74.3, 36.5)
- added Q2: 2N3904BU, Package_TO_SOT_THT:TO-92, F.Cu at (245.7, 122.4)
- added Q3: 2N3904BU, Package_TO_SOT_THT:TO-92, F.Cu at (245.7, 130.0)
- added Q3: 2N3904BU, Package_TO_SOT_THT:TO-92, F.Cu at (244.5, 87.2)
- added Q3: 2N3904BU, Package_TO_SOT_THT:TO-92, F.Cu at (160.2, 88.3)
- added Q3: 2N3904BU, Package_TO_SOT_THT:TO-92, F.Cu at (74.3, 130.4)
- added Q3: 2N3904BU, Package_TO_SOT_THT:TO-92, F.Cu at (160.6, 44.9)
- added Q3: 2N3904BU, Package_TO_SOT_THT:TO-92, F.Cu at (74.3, 44.1)
- added Q3: 2N3904BU, Package_TO_SOT_THT:TO-92, F.Cu at (155.2, 179.3)
- added Q3: 2N3904BU, Package_TO_SOT_THT:TO-92, F.Cu at (159.8, 130.8)
- added Q3: 2N3904BU, Package_TO_SOT_THT:TO-92, F.Cu at (74.3, 88.0)
- added Q3: 2N3904BU, Package_TO_SOT_THT:TO-92, F.Cu at (246.0, 43.8)
- added Q3: 2N3904BU, Package_TO_SOT_THT:TO-92, F.Cu at (73.2, 177.2)
- added Q4: 2N3904BU, Package_TO_SOT_THT:TO-92, F.Cu at (246.0, 51.4)
- added Q4: 2N3904BU, Package_TO_SOT_THT:TO-92, F.Cu at (74.3, 51.8)
- added Q4: 2N3904BU, Package_TO_SOT_THT:TO-92, F.Cu at (160.2, 96.0)
- added Q4: 2N3904BU, Package_TO_SOT_THT:TO-92, F.Cu at (73.2, 184.9)
- added Q4: 2N3904BU, Package_TO_SOT_THT:TO-92, F.Cu at (245.7, 137.6)
- added Q4: 2N3904BU, Package_TO_SOT_THT:TO-92, F.Cu at (155.2, 186.9)
- added Q4: 2N3904BU, Package_TO_SOT_THT:TO-92, F.Cu at (159.8, 138.4)
- added Q4: 2N3904BU, Package_TO_SOT_THT:TO-92, F.Cu at (74.3, 138.0)
- added Q4: 2N3904BU, Package_TO_SOT_THT:TO-92, F.Cu at (74.3, 95.6)
- added Q4: 2N3904BU, Package_TO_SOT_THT:TO-92, F.Cu at (160.6, 52.5)
- added Q4: 2N3904BU, Package_TO_SOT_THT:TO-92, F.Cu at (244.5, 94.8)
- added R1: R_US, Resistor_THT:R_Axial_DIN0207_L6.3mm_D2.5mm_P15.24mm_Horizontal, F.Cu at (54.7, 165.2)
- added R1: R_US, Resistor_THT:R_Axial_DIN0207_L6.3mm_D2.5mm_P15.24mm_Horizontal, F.Cu at (227.6, 31.8)
- added R1: R_US, Resistor_THT:R_Axial_DIN0207_L6.3mm_D2.5mm_P15.24mm_Horizontal, F.Cu at (55.9, 32.1)
- added R1: R_US, Resistor_THT:R_Axial_DIN0207_L6.3mm_D2.5mm_P15.24mm_Horizontal, F.Cu at (55.9, 75.9)
- added R1: R_US, Resistor_THT:R_Axial_DIN0207_L6.3mm_D2.5mm_P15.24mm_Horizontal, F.Cu at (55.9, 118.4)
- added R1: R_US, Resistor_THT:R_Axial_DIN0207_L6.3mm_D2.5mm_P15.24mm_Horizontal, F.Cu at (142.1, 32.9)
- added R1: R_US, Resistor_THT:R_Axial_DIN0207_L6.3mm_D2.5mm_P15.24mm_Horizontal, F.Cu at (136.8, 167.3)
- added R1: R_US, Resistor_THT:R_Axial_DIN0207_L6.3mm_D2.5mm_P15.24mm_Horizontal, F.Cu at (141.4, 118.7)
- added R1: R_US, Resistor_THT:R_Axial_DIN0207_L6.3mm_D2.5mm_P15.24mm_Horizontal, F.Cu at (226.1, 75.2)
- added R1: R_US, Resistor_THT:R_Axial_DIN0207_L6.3mm_D2.5mm_P15.24mm_Horizontal, F.Cu at (141.7, 76.3)
- added R1: R_US, Resistor_THT:R_Axial_DIN0207_L6.3mm_D2.5mm_P15.24mm_Horizontal, F.Cu at (227.2, 118.0)
- added R2: R_US, Resistor_THT:R_Axial_DIN0207_L6.3mm_D2.5mm_P15.24mm_Horizontal, F.Cu at (141.9, 169.8)
- added R2: R_US, Resistor_THT:R_Axial_DIN0207_L6.3mm_D2.5mm_P15.24mm_Horizontal, F.Cu at (232.7, 34.3)
- added R2: R_US, Resistor_THT:R_Axial_DIN0207_L6.3mm_D2.5mm_P15.24mm_Horizontal, F.Cu at (146.8, 78.9)
- added R2: R_US, Resistor_THT:R_Axial_DIN0207_L6.3mm_D2.5mm_P15.24mm_Horizontal, F.Cu at (147.2, 35.4)
- added R2: R_US, Resistor_THT:R_Axial_DIN0207_L6.3mm_D2.5mm_P15.24mm_Horizontal, F.Cu at (61.0, 34.7)
- added R2: R_US, Resistor_THT:R_Axial_DIN0207_L6.3mm_D2.5mm_P15.24mm_Horizontal, F.Cu at (231.1, 77.7)
- added R2: R_US, Resistor_THT:R_Axial_DIN0207_L6.3mm_D2.5mm_P15.24mm_Horizontal, F.Cu at (146.4, 121.3)
- added R2: R_US, Resistor_THT:R_Axial_DIN0207_L6.3mm_D2.5mm_P15.24mm_Horizontal, F.Cu at (61.0, 120.9)
- added R2: R_US, Resistor_THT:R_Axial_DIN0207_L6.3mm_D2.5mm_P15.24mm_Horizontal, F.Cu at (232.3, 120.5)
- added R2: R_US, Resistor_THT:R_Axial_DIN0207_L6.3mm_D2.5mm_P15.24mm_Horizontal, F.Cu at (61.0, 78.5)
- added R2: R_US, Resistor_THT:R_Axial_DIN0207_L6.3mm_D2.5mm_P15.24mm_Horizontal, F.Cu at (59.8, 167.8)
- added R3: R_US, Resistor_THT:R_Axial_DIN0207_L6.3mm_D2.5mm_P15.24mm_Horizontal, F.Cu at (136.7, 73.8)
- added R3: R_US, Resistor_THT:R_Axial_DIN0207_L6.3mm_D2.5mm_P15.24mm_Horizontal, F.Cu at (137.0, 30.4)
- added R3: R_US, Resistor_THT:R_Axial_DIN0207_L6.3mm_D2.5mm_P15.24mm_Horizontal, F.Cu at (222.1, 115.4)
- added R3: R_US, Resistor_THT:R_Axial_DIN0207_L6.3mm_D2.5mm_P15.24mm_Horizontal, F.Cu at (50.8, 29.6)
- added R3: R_US, Resistor_THT:R_Axial_DIN0207_L6.3mm_D2.5mm_P15.24mm_Horizontal, F.Cu at (49.7, 162.7)
- added R3: R_US, Resistor_THT:R_Axial_DIN0207_L6.3mm_D2.5mm_P15.24mm_Horizontal, F.Cu at (50.8, 115.8)
- added R3: R_US, Resistor_THT:R_Axial_DIN0207_L6.3mm_D2.5mm_P15.24mm_Horizontal, F.Cu at (222.5, 29.2)
- added R3: R_US, Resistor_THT:R_Axial_DIN0207_L6.3mm_D2.5mm_P15.24mm_Horizontal, F.Cu at (136.3, 116.2)
- added R3: R_US, Resistor_THT:R_Axial_DIN0207_L6.3mm_D2.5mm_P15.24mm_Horizontal, F.Cu at (221.0, 72.6)
- added R3: R_US, Resistor_THT:R_Axial_DIN0207_L6.3mm_D2.5mm_P15.24mm_Horizontal, F.Cu at (131.7, 164.7)
- added R3: R_US, Resistor_THT:R_Axial_DIN0207_L6.3mm_D2.5mm_P15.24mm_Horizontal, F.Cu at (50.8, 73.4)
- added R4: R_US, Resistor_THT:R_Axial_DIN0207_L6.3mm_D2.5mm_P15.24mm_Horizontal, F.Cu at (131.2, 111.1)
- added R4: R_US, Resistor_THT:R_Axial_DIN0207_L6.3mm_D2.5mm_P15.24mm_Horizontal, F.Cu at (126.6, 159.6)
- added R4: R_US, Resistor_THT:R_Axial_DIN0207_L6.3mm_D2.5mm_P15.24mm_Horizontal, F.Cu at (44.6, 157.6)
- added R4: R_US, Resistor_THT:R_Axial_DIN0207_L6.3mm_D2.5mm_P15.24mm_Horizontal, F.Cu at (217.0, 110.4)
- added R4: R_US, Resistor_THT:R_Axial_DIN0207_L6.3mm_D2.5mm_P15.24mm_Horizontal, F.Cu at (131.6, 68.7)
- added R4: R_US, Resistor_THT:R_Axial_DIN0207_L6.3mm_D2.5mm_P15.24mm_Horizontal, F.Cu at (45.7, 24.5)
- added R4: R_US, Resistor_THT:R_Axial_DIN0207_L6.3mm_D2.5mm_P15.24mm_Horizontal, F.Cu at (45.7, 68.3)
- added R4: R_US, Resistor_THT:R_Axial_DIN0207_L6.3mm_D2.5mm_P15.24mm_Horizontal, F.Cu at (132.0, 25.3)
- added R4: R_US, Resistor_THT:R_Axial_DIN0207_L6.3mm_D2.5mm_P15.24mm_Horizontal, F.Cu at (215.9, 67.6)
- added R4: R_US, Resistor_THT:R_Axial_DIN0207_L6.3mm_D2.5mm_P15.24mm_Horizontal, F.Cu at (217.4, 24.1)
- added R4: R_US, Resistor_THT:R_Axial_DIN0207_L6.3mm_D2.5mm_P15.24mm_Horizontal, F.Cu at (45.7, 110.7)
- added U1: 4017, Package_DIP:DIP-16_W7.62mm_Socket_LongPads, F.Cu at (40.6, 93.7)
- added U1: 4017, Package_DIP:DIP-16_W7.62mm_Socket_LongPads, F.Cu at (210.8, 93.0)
- added U1: 4017, Package_DIP:DIP-16_W7.62mm_Socket_LongPads, F.Cu at (126.9, 50.7)
- added U1: 4017, Package_DIP:DIP-16_W7.62mm_Socket_LongPads, F.Cu at (39.5, 183.0)
- added U1: 4017, Package_DIP:DIP-16_W7.62mm_Socket_LongPads, F.Cu at (40.6, 136.1)
- added U1: 4017, Package_DIP:DIP-16_W7.62mm_Socket_LongPads, F.Cu at (212.0, 135.8)
- added U1: 4017, Package_DIP:DIP-16_W7.62mm_Socket_LongPads, F.Cu at (121.5, 185.0)
- added U1: 4017, Package_DIP:DIP-16_W7.62mm_Socket_LongPads, F.Cu at (40.6, 49.9)
- added U1: 4017, Package_DIP:DIP-16_W7.62mm_Socket_LongPads, F.Cu at (212.3, 49.5)
- added U1: 4017, Package_DIP:DIP-16_W7.62mm_Socket_LongPads, F.Cu at (126.1, 136.5)
- added U1: 4017, Package_DIP:DIP-16_W7.62mm_Socket_LongPads, F.Cu at (126.5, 94.1)
Routing:
- net GND: track 0.00 -> 2217.8 mm
- net Net-(Q4-Pad2): track 0.00 -> 486.2 mm
- net Net-(Q3-Pad2): track 0.00 -> 333.5 mm
- net +5V: track 0.00 -> 309.3 mm
- net Net-(Q1-Pad2): track 0.00 -> 249.2 mm
- net Net-(R2-Pad2): track 0.00 -> 235.1 mm
- net Net-(U1-Pad10): track 0.00 -> 218.7 mm
- net Net-(R1-Pad2): track 0.00 -> 179.2 mm
- net Net-(Q2-Pad2): track 0.00 -> 170.1 mm
- net Net-(J1-Pad4): track 0.00 -> 134.9 mm
- net Net-(J1-Pad1): track 0.00 -> 123.3 mm
- net Net-(R3-Pad2): track 0.00 -> 123.3 mm
- net Net-(J1-Pad3): track 0.00 -> 116.2 mm
- net Net-(J1-Pad2): track 0.00 -> 111.8 mm
- net /555_signal: track 0.00 -> 95.4 mm
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Other:
- board outline added: 250.6 x 175.1 mm
