File: Generador de señales/Generador de señales.kicad_sch (KiCad schematic)
At the start: 6 parts, among them J1 Conn_01x03, U1 NA555P

Commit message: final
Parts:
- C1: footprint (none) -> Capacitor_THT:CP_Radial_D7.5mm_P2.50mm
- C2: footprint (none) -> Capacitor_THT:C_Disc_D3.0mm_W1.6mm_P2.50mm
- J1: footprint (none) -> TerminalBlock:TerminalBlock_bornier-3_P5.08mm
- R1, R2: footprint (none) -> Resistor_THT:R_Axial_DIN0204_L3.6mm_D1.6mm_P5.08mm_Horizontal
Changed lines of the file:
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@@
   (symbol (lib_id "power:GND") (at 92.71 71.12 0) (unit 1)
     (in_bom yes) (on_board yes)
-    (property "Reference" "#PWR?" (id 0) (at 92.71 77.47 0)
+    (property "Reference" "#PWR0106" (id 0) (at 92.71 77.47 0)
       (effects (font (size 1 1)) hide)
     )
@@
   (symbol (lib_id "power:GND") (at 76.2 119.38 0) (unit 1)
     (in_bom yes) (on_board yes)
-    (property "Reference" "#PWR?" (id 0) (at 76.2 125.73 0)
+    (property "Reference" "#PWR0103" (id 0) (at 76.2 125.73 0)
       (effects (font (size 1 1)) hide)
     )
@@
   (symbol (lib_id "power:+5V") (at 90.17 71.12 180) (unit 1)
     (in_bom yes) (on_board yes) (fields_autoplaced)
-    (property "Reference" "#PWR?" (id 0) (at 90.17 67.31 0)
+    (property "Reference" "#PWR0104" (id 0) (at 90.17 67.31 0)
       (effects (font (size 1 1)) hide)
     )
@@
   (symbol (lib_id "power:GND") (at 36.83 106.68 270) (unit 1)
     (in_bom yes) (on_board yes)
-    (property "Reference" "#PWR?" (id 0) (at 30.48 106.68 0)
+    (property "Reference" "#PWR0108" (id 0) (at 30.48 106.68 0)
       (effects (font (size 1 1)) hide)
     )
@@
   (symbol (lib_id "power:GND") (at 63.5 116.84 0) (unit 1)
     (in_bom yes) (on_board yes)
-    (property "Reference" "#PWR?" (id 0) (at 63.5 123.19 0)
+    (property "Reference" "#PWR0102" (id 0) (at 63.5 123.19 0)
       (effects (font (size 1 1)) hide)
     )
@@
   (symbol (lib_id "power:+5V") (at 92.71 106.68 270) (unit 1)
     (in_bom yes) (on_board yes) (fields_autoplaced)
-    (property "Reference" "#PWR?" (id 0) (at 88.9 106.68 0)
+    (property "Reference" "#PWR0105" (id 0) (at 88.9 106.68 0)
       (effects (font (size 1 1)) hide)
     )
@@
     (property "Reference" "C2" (id 0) (at 30.48 113.03 90))
     (property "Value" "C_Polarized_US" (id 1) (at 30.48 110.49 90))
-    (property "Footprint" "" (id 2) (at 40.64 106.68 0)
+    (property "Footprint" "Capacitor_THT:C_Disc_D3.0mm_W1.6mm_P2.50mm" (id 2) (at 40.64 106.68 0)
       (effects (font (size 1.27 1.27)) hide)
     )
@@
       (effects (font (size 1.27 1.27)) (justify left))
     )
-    (property "Footprint" "" (id 2) (at 76.2 115.57 0)
+    (property "Footprint" "Capacitor_THT:CP_Radial_D7.5mm_P2.50mm" (id 2) (at 76.2 115.57 0)
       (effects (font (size 1.27 1.27)) hide)
     )
@@
       (effects (font (size 1 1)) (justify right))
     )
-    (property "Footprint" "" (id 2) (at 92.71 66.04 0)
+    (property "Footprint" "TerminalBlock:TerminalBlock_bornier-3_P5.08mm" (id 2) (at 92.71 66.04 0)
       (effects (font (size 1.27 1.27)) hide)
     )
@@
       (effects (font (size 1 1)) (justify left))
     )
-    (property "Footprint" "" (id 2) (at 51.816 92.964 90)
+    (property "Footprint" "Resistor_THT:R_Axial_DIN0204_L3.6mm_D1.6mm_P5.08mm_Horizontal" (id 2) (at 51.816 92.964 90)
       (effects (font (size 1.27 1.27)) hide)
     )
@@
       (effects (font (size 1 1)))
     )
-    (property "Footprint" "" (id 2) (at 89.154 105.664 90)
+    (property "Footprint" "Resistor_THT:R_Axial_DIN0204_L3.6mm_D1.6mm_P5.08mm_Horizontal" (id 2) (at 89.154 105.664 90)
       (effects (font (size 1.27 1.27)) hide)
     )
@@
   (symbol (lib_id "power:+5V") (at 50.8 111.76 90) (unit 1)
     (in_bom yes) (on_board yes)
-    (property "Reference" "#PWR?" (id 0) (at 54.61 111.76 0)
+    (property "Reference" "#PWR0107" (id 0) (at 54.61 111.76 0)
       (effects (font (size 1 1)) hide)
     )
@@
   (symbol (lib_id "power:+5V") (at 63.5 96.52 0) (unit 1)
     (in_bom yes) (on_board yes)
-    (property "Reference" "#PWR?" (id 0) (at 63.5 100.33 0)
+    (property "Reference" "#PWR0101" (id 0) (at 63.5 100.33 0)
       (effects (font (size 1 1)) hide)
     )
@@
   )
   (symbol_instances
+    (path "/dc1793c3-db23-46e9-8a11-cde7fe8a1ca5"
+      (reference "#PWR0101") (unit 1) (value "+5V") (footprint "")
+    )
+    (path "/2f1a9ef1-daff-4fd8-bcb5-1aaf1512479e"
+      (reference "#PWR0102") (unit 1) (value "GND") (footprint "")
+    )
+    (path "/0c5b61d0-df61-4bbd-abd4-6c526dc81fb0"
+      (reference "#PWR0103") (unit 1) (value "GND") (footprint "")
+    )
+    (path "/19991cde-5872-4534-b621-6cbf04dc9f4c"
+      (reference "#PWR0104") (unit 1) (value "+5V") (footprint "")
+    )
+    (path "/5acf282b-2f25-4bd5-8f72-975fd6810597"
+      (reference "#PWR0105") (unit 1) (value "+5V") (footprint "")
+    )
     (path "/09108e89-2eef-4e74-bf52-be838a1dea43"
-      (reference "#PWR?") (unit 1) (value "GND") (footprint "")
-    )
-    (path "/0c5b61d0-df61-4bbd-abd4-6c526dc81fb0"
-      (reference "#PWR?") (unit 1) (value "GND") (footprint "")
-    )
-    (path "/19991cde-5872-4534-b621-6cbf04dc9f4c"
-      (reference "#PWR?") (unit 1) (value "+5V") (footprint "")
+      (reference "#PWR0106") (unit 1) (value "GND") (footprint "")
+    )
+    (path "/a77acde8-9446-4107-b663-4e41b2db6b48"
+      (reference "#PWR0107") (unit 1) (value "+5V") (footprint "")
     )
     (path "/23a983a3-5674-4829-98c2-27172d7b52be"
-      (reference "#PWR?") (unit 1) (value "GND") (footprint "")
-    )
-    (path "/2f1a9ef1-daff-4fd8-bcb5-1aaf1512479e"
-      (reference "#PWR?") (unit 1) (value "GND") (footprint "")
-    )
-    (path "/5acf282b-2f25-4bd5-8f72-975fd6810597"
-      (reference "#PWR?") (unit 1) (value "+5V") (footprint "")
-    )
-    (path "/a77acde8-9446-4107-b663-4e41b2db6b48"
-      (reference "#PWR?") (unit 1) (value "+5V") (footprint "")
-    )
-    (path "/dc1793c3-db23-46e9-8a11-cde7fe8a1ca5"
-      (reference "#PWR?") (unit 1) (value "+5V") (footprint "")
+      (reference "#PWR0108") (unit 1) (value "GND") (footprint "")
     )
     (path "/709be9fe-baec-414c-ac10-e2d420363d94"
-      (reference "C1") (unit 1) (value "C_Polarized_US") (footprint "")
+      (reference "C1") (unit 1) (value "C_Polarized_US") (footprint "Capacitor_THT:CP_Radial_D7.5mm_P2.50mm")
     )
     (path "/708fad39-06c7-4f90-a5b4-ccefab4d7bc6"
-      (reference "C2") (unit 1) (value "C_Polarized_US") (footprint "")
+      (reference "C2") (unit 1) (value "C_Polarized_US") (footprint "Capacitor_THT:C_Disc_D3.0mm_W1.6mm_P2.50mm")
     )
     (path "/7d460f2d-be21-48d4-8c62-dcddd19d1a5d"
-      (reference "J1") (unit 1) (value "Conn_01x03") (footprint "")
+      (reference "J1") (unit 1) (value "Conn_01x03") (footprint "TerminalBlock:TerminalBlock_bornier-3_P5.08mm")
     )
     (path "/920418c3-c219-44ea-8bea-fb3407c67f4c"
-      (reference "R1") (unit 1) (value "R_US") (footprint "")
+      (reference "R1") (unit 1) (value "R_US") (footprint "Resistor_THT:R_Axial_DIN0204_L3.6mm_D1.6mm_P5.08mm_Horizontal")
     )
     (path "/a57de01d-930a-4463-9411-c6e7a2020687"
-      (reference "R2") (unit 1) (value "R_US") (footprint "")
+      (reference "R2") (unit 1) (value "R_US") (footprint "Resistor_THT:R_Axial_DIN0204_L3.6mm_D1.6mm_P5.08mm_Horizontal")
     )
     (path "/0fb27e11-fde6-4a25-adbb-e9684771b369"
